Commit message: working on hotspray motion

File: hotspray_description/urdf/coil.urdf (robot description, URDF)
Before this commit: robot coil, 2 links, 1 joints
Links:
- link base: geometry collision box size=0.4 0.4 0.01
- link coil: geometry collision mesh filename=package://hotspray_description/meshes/coil.stl scale=0.001 0.001 0.001; visual mesh filename=package://hotspray_description/meshes/coil.stl scale=0.001 0.001 0.001

Commit message: refactoring

File: hotspray_description/urdf/coil.urdf (robot description, URDF)
Before this commit: robot coil, 2 links, 1 joints
Links:
- link coil: geometry visual mesh filename=package://hotspray_description/meshes/coil.stl scale=0.0009 0.0009 0.0009

File: hotspray_description/urdf/hotspray_application.xacro (robot description, xacro)
@@ -2,5 +2,5 @@
 <robot xmlns:xacro="http://www.ros.org/wiki/xacro" name="hotspray_description">
   <xacro:property name="sim" default="true"/>
-  <xacro:property name="joint_limited" default="true"/>
+  <xacro:property name="joint_limited" default="false"/>
   <xacro:property name="prefix" value=""/>
   <xacro:arg name="transmission_hw_interface" default="hardware_interface/PositionJointInterface" />
@@ -8,10 +8,9 @@
   <xacro:include filename="$(find hotspray_description)/urdf/hotspray_workcell.xacro"/>
   <xacro:include filename="$(find ur_description)/urdf/ur5.urdf.xacro" />
-  <!-- <xacro:include filename="$(find tesseract_ros_examples)/urdf/lbr_iiwa_14_r820_macro.xacro" /> -->
-  <!-- robot -->
+  <xacro:property name="deg_to_rad" value="0.01745329251994329577" />
+    <!-- robot -->
     <xacro:if value="${sim}">
         <xacro:include filename="$(find ur_description)/urdf/common.gazebo.xacro" />
     </xacro:if>
-    <!-- arm -->
     <xacro:if value="${joint_limited}">
       <xacro:ur5_robot prefix="${prefix}" joint_limited="true"
@@ -26,11 +25,27 @@
     </xacro:if>
     <xacro:unless value="${joint_limited}">
-        <xacro:ur5_robot prefix="${prefix}" joint_limited="false"
-          transmission_hw_interface="$(arg transmission_hw_interface)"
-        />
+      <xacro:ur5_robot prefix="${prefix}" joint_limited="true"
+        shoulder_pan_lower_limit="0.0" shoulder_pan_upper_limit="3.12414"
+        shoulder_lift_lower_limit="-2.26893" shoulder_lift_upper_limit="-0.523599"
+        elbow_joint_lower_limit="${-2*pi}" elbow_joint_upper_limit="${2*pi}"
+        wrist_1_lower_limit="-4.01426" wrist_1_upper_limit="0.785398"
+        wrist_2_lower_limit="-4.01426" wrist_2_upper_limit="0.785398"
+        wrist_3_lower_limit="${-2*pi}" wrist_3_upper_limit="${2*pi}"
+        transmission_hw_interface="$(arg transmission_hw_interface)"
+      />
     </xacro:unless>
-      <!-- <xacro:kuka_lbr_iiwa_14_r820 prefix=""/> -->
-  <!-- link world->robot -->
-   <link name="world"/>
+    <!-- <xacro:unless value="${joint_limited}">
+      <xacro:ur5_robot prefix="${prefix}" joint_limited="true"
+        shoulder_pan_lower_limit="${-2*pi}" shoulder_pan_upper_limit="${2*pi}"
+        shoulder_lift_lower_limit="${-2*pi}" shoulder_lift_upper_limit="${2*pi}"
+        elbow_joint_lower_limit="${-2*pi}" elbow_joint_upper_limit="${2*pi}"
+        wrist_1_lower_limit="${-2*pi}" wrist_1_upper_limit="${2*pi}"
+        wrist_2_lower_limit="${-2*pi}" wrist_2_upper_limit="${2*pi}"
+        wrist_3_lower_limit="${-2*pi}" wrist_3_upper_limit="${2*pi}"
+        transmission_hw_interface="$(arg transmission_hw_interface)"
+      />
+    </xacro:unless> -->
+  <!-- link world-robot -->
+    <link name="world"/>
       <joint name="world_to_robot" type="fixed">
       <parent link="world"/>
@@ -40,5 +55,5 @@
   <!-- table -->
     <xacro:hotspray_workcell parent="world">
-      <origin  xyz="0 0 0" rpy="0 0 0" />
+      <origin  xyz="0 0 0" rpy="0 0 0" />3
     </xacro:hotspray_workcell>
   <!-- scan area -->
@@ -49,7 +64,7 @@
       <origin  xyz="0.2 0.2 0.55" rpy="0 0 0" />
     </joint>
-  <!-- tool  -->
+  <!-- tool -->
     <xacro:hotspray_tool parent="tool0" prefix="${prefix}" sim="${sim}">
-      <origin  xyz="0 0 0" rpy="0 0 ${pi/4}" />
+      <origin  xyz="0 0 0.0" rpy="0 0 0" />
     </xacro:hotspray_tool>
 </robot>

File: hotspray_description/urdf/hotspray_extruder.xacro (robot description, xacro)
@@ -1,14 +1,22 @@
 <?xml version="1.0" ?>
 <robot xmlns:xacro="http://www.ros.org/wiki/xacro">
+  <!-- <xacro:property name="deg_to_rad" value="0.01745329251994329577" /> -->
   <xacro:macro name="hotspray_extruder" params="parent *origin spray_distance:=${'10.0'}">
+      <!-- extruder_link -->
+    <link name="extruder_link"/>
+      <joint name="extruder_link_joint" type="fixed">
+        <parent link="${parent}"/>
+      <child link="extruder_link"/>
+        <xacro:insert_block name="origin"/>
+      </joint>
     <link name="hotspray_extruder">
       <!-- TODO: inertia hotspray-->
       <inertial>
-        <origin  xyz="0 0 0" rpy="0 0 0" />
-        <mass value="0" />
-        <inertia ixx="0.00" ixy="0" ixz="0" iyy="0.00" iyz="0" izz="0.00" />
+        <origin  xyz="0.0 0.0 0.0" rpy="0.0 0.0 0.0" />
+        <mass value="0.0" />
+        <inertia ixx="0.0" ixy="0.0" ixz="0.0" iyy="0.0" iyz="0.0" izz="0.0" />
       </inertial>
       <visual>
-        <origin  xyz="0 0 0" rpy="0 0 0" />
+        <origin  xyz="0 0 0" rpy="0 ${-pi/2} ${pi/2}" />
         <geometry>
           <mesh filename="package://hotspray_description/meshes/hotspray_extruder.stl" scale="0.001 0.001 0.001" />
@@ -18,16 +26,36 @@
         </material>
       </visual>
-      <!--collision>
+      <collision>
+        <origin  xyz="-0.015 0.0 0.01" rpy="0.0 0.0 0.0" />
+        <geometry>
+          <box size="0.04 0.11 0.11"/>
+        </geometry>
+      </collision>
+      </link>
+      <link name="hotspray_extruder_hose_collission">
+        <collision>
+          <origin  xyz="-0.015 0.13 -0.01" rpy="${pi/2} 0.0 0.0" />
+          <geometry>
+            <cylinder length="0.15" radius="0.02"/>
+          </geometry>
+        </collision>
+      </link>
+      <joint name="hotspray_extruder_hose_collission_joint" type="fixed">
+        <parent link="${parent}" />
+      <child link="hotspray_extruder_hose_collission" />
         <xacro:insert_block name="origin"/>
-        <geometry>
-          <box size="0.195 0.04 0.27"/>
-        </geometry>
-      </collision-->
-    </link>
-    <!--joint between fixture and hotspray-->
-    <joint name="hotspray_extruder_joint" type="fixed">
-      <xacro:insert_block name="origin"/>
-      <parent link="${parent}" />
+      </joint>
+    <!-- joint between fixture and hotspray -->
+      <joint name="hotspray_extruder_joint" type="fixed">
+        <parent link="${parent}" />
       <child link="hotspray_extruder" />
+        <xacro:insert_block name="origin"/>
+      </joint>
+    <!-- tcp_frame -->
+    <link name="tcp_frame"/>
+      <joint name="tcp_frame_joint" type="fixed">
+        <parent link="extruder_link"/>
+      <child link="tcp_frame"/>
+        <origin xyz="-0.01 -0.03 0.16" rpy="0.0 0.0 0.0"/>
     </joint>
   </xacro:macro>

File: hotspray_description/urdf/hotspray_tool.xacro (robot description, xacro)
@@ -1,6 +1,9 @@
 <?xml version="1.0" ?>
 <robot xmlns:xacro="http://www.ros.org/wiki/xacro">
+  <xacro:property name="deg_to_rad" value="0.01745329251994329577" />
   <xacro:macro name="hotspray_tool" params="parent *origin prefix:=${''} sim">
     <xacro:include filename="$(find hotspray_description)/urdf/hotspray_extruder.xacro"/>
+    <xacro:include filename="$(find hotspray_description)/urdf/hotspray_camera.xacro"/>
+    <xacro:property name="deg_to_rad" value="0.01745329251994329577" />
     <link name="hotspray_tool_link"/>
       <joint name="tool_to_ur5_tool0" type="fixed">
@@ -9,33 +12,15 @@
         <xacro:insert_block name="origin"/>
       </joint>
-    <!-- simulated camera -->
-    <xacro:if value="${sim}">
-      <xacro:include filename="$(find hotspray_description)/urdf/camera/_d435.urdf.xacro"/>
-        <xacro:arg name="add_plug" default="false" />
-          <xacro:sensor_d435 parent="hotspray_tool_link" >
-        <origin xyz="-0.02 -0.0175 0.023" rpy="${pi/2} ${-pi/2} ${pi/2}"/>
-      </xacro:sensor_d435>
-    </xacro:if>
-    <!-- real camera -->
-    <xacro:unless value="${sim}">
-      <xacro:include filename="$(find realsense2_description)/urdf/_d435.urdf.xacro" />
-        <xacro:arg name="use_nominal_extrinsics" default="false"/>
-        <xacro:arg name="add_plug" default="false" />
-        <xacro:sensor_d435 parent="hotspray_tool_link" use_nominal_extrinsics="$(arg use_nominal_extrinsics)" add_plug="$(arg add_plug)">
-          <origin xyz="-0.02 -0.0175 0.023" rpy="${pi/2} ${-pi/2} ${pi/2}"/>
-        </xacro:sensor_d435>
-    </xacro:unless>
+    <!-- camera -->
+      <!-- origin xyz="-0.035 -0.07 0.055" rpy="${-pi/2} ${-pi/2} ${pi/2}"  -->
+    <xacro:hotspray_camera parent="hotspray_tool_link" sim="${sim}">
+      <origin xyz="0.03 0.0 0.05" rpy="${pi/2} 0.0 0" />
+    </xacro:hotspray_camera>
     <!-- extruder -->
-      <xacro:hotspray_extruder parent="hotspray_tool_link">
-        <!-- origin xyz="-0.035 -0.07 0.055" rpy="${-pi/2} ${-pi/2} ${pi/2}" /-->
-        <origin xyz="0.12 -0.03 0.04" rpy="0 ${-pi/2} ${pi/2}" />
-      </xacro:hotspray_extruder>
-    <!-- tcp -->
-    <link name="tcp_frame"/>
-      <joint name="tcp_frame_joint" type="fixed">
-        <parent link="tool0"/>
-      <child link="tcp_frame"/>
-        <origin xyz="0.12 0.03 0.16" rpy="0 0 ${pi/4}"/>
-    </joint>
+    <xacro:hotspray_extruder parent="hotspray_tool_link">
+      <!-- <origin xyz="-0.1 -0.04 0.04" rpy="${-2 * pi/3} 0 ${pi}" /> -->
+      <!-- <origin xyz="-0.1 -0.04 0.04" rpy="${-pi/3} 0 ${pi}" /> -->
+      <origin xyz="-0.1 -0.04 0.04" rpy="${-pi/2} 0 ${pi}" />
+    </xacro:hotspray_extruder>
   </xacro:macro>
 </robot>

File: hotspray_description/urdf/hotspray_workcell.xacro (robot description, xacro)
@@ -26,43 +26,43 @@
           </geometry>
         </collision>
-            <inertial>
+    <inertial>
       <mass value="10.0" />
       <inertia  ixx="1.0" ixy="0.0"  ixz="0.0"  iyy="1.0"  iyz="0.0"  izz="1.0" />
     </inertial>
     <!-- top -->
-        <collision>
+        <!-- <collision>
           <origin rpy="0 0 0" xyz="${offset} ${offset} ${table_height + workspace_height + wall_width/2}"/>
           <geometry>
              <box size="${workspace_width} ${workspace_width} ${wall_width}"/>
           </geometry>
-        </collision>
+        </collision> -->
     <!-- front -->
-        <collision>
+        <!-- <collision>
           <origin rpy="0 0 0" xyz="${offset} ${offset - workspace_width/2 - wall_width/2} ${table_height + workspace_height/2}"/>
           <geometry>
              <box size="${workspace_width} ${wall_width} ${workspace_height}"/>
           </geometry>
-        </collision>
+        </collision> -->
     <!-- back -->
-        <collision>
+        <!-- <collision>
           <origin rpy="0 0 0" xyz="${offset} ${offset + workspace_width/2 + wall_width/2} ${table_height + workspace_height/2}"/>
           <geometry>
              <box size="${workspace_width} ${wall_width} ${workspace_height}"/>
           </geometry>
-        </collision>
+        </collision> -->
     <!-- left -->
-        <collision>
+        <!-- <collision>
           <origin rpy="0 0 0" xyz="${offset - workspace_width/2 - wall_width/2} ${offset} ${table_height + workspace_height/2}"/>
           <geometry>
              <box size="${wall_width} ${workspace_width} ${workspace_height}"/>
           </geometry>
-        </collision>
+        </collision> -->
     <!-- right -->
-        <collision>
+        <!-- <collision>
           <origin rpy="0 0 0" xyz="${offset + workspace_width/2 + wall_width/2} ${offset} ${table_height + workspace_height/2}"/>
           <geometry>
              <box size="${wall_width} ${workspace_width} ${workspace_height}"/>
           </geometry>
-        </collision>
+        </collision> -->
     </link>
     <joint name="workcell_joint" type="fixed">
