Commit message: motion

File: hotspray_description/urdf/hotspray_application.xacro (robot description, xacro)
@@ -8,4 +8,5 @@
   <xacro:include filename="$(find hotspray_description)/urdf/hotspray_workcell.xacro"/>
   <xacro:include filename="$(find ur_description)/urdf/ur5.urdf.xacro" />
+  <xacro:include filename="$(find ur_description)/urdf/ur5.urdf.xacro" />
   <xacro:property name="deg_to_rad" value="0.01745329251994329577" />
     <!-- robot -->
@@ -15,18 +16,7 @@
     <xacro:if value="${joint_limited}">
       <xacro:ur5_robot prefix="${prefix}" joint_limited="true"
-        shoulder_pan_lower_limit="${-pi}" shoulder_pan_upper_limit="${pi}"
-        shoulder_lift_lower_limit="${-pi}" shoulder_lift_upper_limit="${pi}"
-        elbow_joint_lower_limit="${-pi}" elbow_joint_upper_limit="${pi}"
-        wrist_1_lower_limit="${-pi}" wrist_1_upper_limit="${pi}"
-        wrist_2_lower_limit="${-pi}" wrist_2_upper_limit="${pi}"
-        wrist_3_lower_limit="${-pi}" wrist_3_upper_limit="${pi}"
-        transmission_hw_interface="$(arg transmission_hw_interface)"
-      />
-    </xacro:if>
-    <xacro:unless value="${joint_limited}">
-      <xacro:ur5_robot prefix="${prefix}" joint_limited="true"
         shoulder_pan_lower_limit="0.0" shoulder_pan_upper_limit="3.12414"
         shoulder_lift_lower_limit="-2.26893" shoulder_lift_upper_limit="-0.523599"
-        elbow_joint_lower_limit="${-2*pi}" elbow_joint_upper_limit="${2*pi}"
+        elbow_joint_lower_limit="-0.523599" elbow_joint_upper_limit="2.79253"
         wrist_1_lower_limit="-4.01426" wrist_1_upper_limit="0.785398"
         wrist_2_lower_limit="-4.01426" wrist_2_upper_limit="0.785398"
@@ -34,6 +24,6 @@
         transmission_hw_interface="$(arg transmission_hw_interface)"
       />
-    </xacro:unless>
-    <!-- <xacro:unless value="${joint_limited}">
+    </xacro:if>
+    <xacro:unless value="${joint_limited}">
       <xacro:ur5_robot prefix="${prefix}" joint_limited="true"
         shoulder_pan_lower_limit="${-2*pi}" shoulder_pan_upper_limit="${2*pi}"
@@ -45,10 +35,10 @@
         transmission_hw_interface="$(arg transmission_hw_interface)"
       />
-    </xacro:unless> -->
+    </xacro:unless>
   <!-- link world-robot -->
     <link name="world"/>
       <joint name="world_to_robot" type="fixed">
-      <parent link="world"/>
-      <child link="base_link"/>
+        <parent link="world"/>
+        <child link="base_link"/>
       <origin  xyz="0 0 0.501" rpy="0 0 ${7 * pi/4}" />
     </joint>
@@ -60,7 +50,7 @@
     <link name="tsdf_origin"/>
       <joint name="world_to_tsdf" type="fixed">
-      <parent link="world"/>
-      <child link="tsdf_origin"/>
-      <origin  xyz="0.2 0.2 0.55" rpy="0 0 0" />
+        <parent link="world"/>
+        <child link="tsdf_origin"/>
+      <origin  xyz="0.25 0.25 0.55" rpy="0 0 0" />
     </joint>
   <!-- tool -->
@@ -68,3 +58,10 @@
       <origin  xyz="0 0 0.0" rpy="0 0 0" />
     </xacro:hotspray_tool>
+  <!-- coil -->
+    <xacro:if value="${sim}">
+    <xacro:include filename="$(find hotspray_description)/urdf/coil_fixed.xacro"/>
+      <xacro:coil parent="base_link">
+        <origin  xyz="0.0 0.6 0.1" rpy="0 0 0.0" />
+      </xacro:coil>
+    </xacro:if>
 </robot>

File: hotspray_description/urdf/hotspray_camera.xacro (robot description, xacro)
@@ -24,5 +24,5 @@
         <parent link="camera_link"/>
       <child link="camera_orbit_frame"/>
-        <origin xyz="0.25 0.0 0.0" rpy="${5* pi/6} ${-pi/2} 0"/>
+        <origin xyz="0.25 0.0 0.0" rpy="${-pi/4} ${-pi/2} 0"/>
     </joint>
   </xacro:macro>

File: hotspray_description/urdf/hotspray_extruder.xacro (robot description, xacro)
@@ -2,5 +2,5 @@
 <robot xmlns:xacro="http://www.ros.org/wiki/xacro">
   <!-- <xacro:property name="deg_to_rad" value="0.01745329251994329577" /> -->
-  <xacro:macro name="hotspray_extruder" params="parent *origin spray_distance:=${'10.0'}">
+  <xacro:macro name="hotspray_extruder" params="parent *origin spray_distance:=${'0.1'}">
       <!-- extruder_link -->
     <link name="extruder_link"/>
@@ -11,5 +11,4 @@
       </joint>
     <link name="hotspray_extruder">
-      <!-- TODO: inertia hotspray-->
       <inertial>
         <origin  xyz="0.0 0.0 0.0" rpy="0.0 0.0 0.0" />
@@ -33,5 +32,5 @@
       </collision>
       </link>
-      <link name="hotspray_extruder_hose_collission">
+      <!-- <link name="hotspray_extruder_hose_collission">
         <collision>
           <origin  xyz="-0.015 0.13 -0.01" rpy="${pi/2} 0.0 0.0" />
@@ -40,12 +39,12 @@
           </geometry>
         </collision>
-      </link>
-      <joint name="hotspray_extruder_hose_collission_joint" type="fixed">
+      </link> -->
+      <!-- <joint name="hotspray_extruder_hose_collission_joint" type="fixed">
         <parent link="${parent}" />
       <child link="hotspray_extruder_hose_collission" />
         <xacro:insert_block name="origin"/>
-      </joint>
+      </joint> -->
     <!-- joint between fixture and hotspray -->
-      <joint name="hotspray_extruder_joint" type="fixed">
+       <joint name="hotspray_extruder_joint" type="fixed">
         <parent link="${parent}" />
       <child link="hotspray_extruder" />
@@ -57,5 +56,5 @@
         <parent link="extruder_link"/>
       <child link="tcp_frame"/>
-        <origin xyz="-0.01 -0.03 0.16" rpy="0.0 0.0 0.0"/>
+        <origin xyz="-0.01 -0.03 ${spray_distance}" rpy="0.0 0.0 0.0"/>
     </joint>
   </xacro:macro>

File: hotspray_description/urdf/hotspray_tool.xacro (robot description, xacro)
@@ -15,13 +15,17 @@
       <!-- origin xyz="-0.035 -0.07 0.055" rpy="${-pi/2} ${-pi/2} ${pi/2}"  -->
     <xacro:hotspray_camera parent="hotspray_tool_link" sim="${sim}">
-      <origin xyz="0.03 0.0 0.05" rpy="${pi/2} 0.0 0" />
+      <origin xyz="0.03 0.0 0.05" rpy="${pi/2} ${-pi/4} 0" />
     </xacro:hotspray_camera>
     <!-- extruder -->
     <xacro:hotspray_extruder parent="hotspray_tool_link">
+      <!-- in -120 degree up facing -->
       <!-- <origin xyz="-0.1 -0.04 0.04" rpy="${-2 * pi/3} 0 ${pi}" /> -->
+      <!-- in -60 degree down facing -->
       <!-- <origin xyz="-0.1 -0.04 0.04" rpy="${-pi/3} 0 ${pi}" /> -->
+      <!-- in y direction -->
       <origin xyz="-0.1 -0.04 0.04" rpy="${-pi/2} 0 ${pi}" />
+      <!-- in z direction -->
+      <!-- <origin xyz="-0.1 -0.04 0.04" rpy="0 0 ${pi}" /> -->
     </xacro:hotspray_extruder>
-IOStates
   </xacro:macro>
 </robot>

File: hotspray_description/urdf/hotspray_workcell.xacro (robot description, xacro)
@@ -26,43 +26,51 @@
           </geometry>
         </collision>
-    <inertial>
-      <mass value="10.0" />
-      <inertia  ixx="1.0" ixy="0.0"  ixz="0.0"  iyy="1.0"  iyz="0.0"  izz="1.0" />
-    </inertial>
+        <inertial>
+          <mass value="10.0" />
+          <inertia  ixx="1.0" ixy="0.0"  ixz="0.0"  iyy="1.0"  iyz="0.0"  izz="1.0" />
+        </inertial>
     <!-- top -->
-        <!-- <collision>
+        <collision>
           <origin rpy="0 0 0" xyz="${offset} ${offset} ${table_height + workspace_height + wall_width/2}"/>
           <geometry>
              <box size="${workspace_width} ${workspace_width} ${wall_width}"/>
           </geometry>
-        </collision> -->
+        </collision>
     <!-- front -->
-        <!-- <collision>
+        <collision>
           <origin rpy="0 0 0" xyz="${offset} ${offset - workspace_width/2 - wall_width/2} ${table_height + workspace_height/2}"/>
           <geometry>
              <box size="${workspace_width} ${wall_width} ${workspace_height}"/>
           </geometry>
-        </collision> -->
+        </collision>
     <!-- back -->
-        <!-- <collision>
+        <collision>
           <origin rpy="0 0 0" xyz="${offset} ${offset + workspace_width/2 + wall_width/2} ${table_height + workspace_height/2}"/>
           <geometry>
              <box size="${workspace_width} ${wall_width} ${workspace_height}"/>
           </geometry>
-        </collision> -->
+        </collision>
     <!-- left -->
-        <!-- <collision>
+        <collision>
           <origin rpy="0 0 0" xyz="${offset - workspace_width/2 - wall_width/2} ${offset} ${table_height + workspace_height/2}"/>
           <geometry>
              <box size="${wall_width} ${workspace_width} ${workspace_height}"/>
           </geometry>
-        </collision> -->
+        </collision>
     <!-- right -->
-        <!-- <collision>
+        <collision>
           <origin rpy="0 0 0" xyz="${offset + workspace_width/2 + wall_width/2} ${offset} ${table_height + workspace_height/2}"/>
           <geometry>
              <box size="${wall_width} ${workspace_width} ${workspace_height}"/>
           </geometry>
-        </collision> -->
+        </collision>
+    <!-- rotation table collision-->
+        <xacro:property name="rotation_table_height" value="0.1"/>
+        <collision>
+          <origin rpy="0 0 0" xyz="0.35 0.35 ${table_height + rotation_table_height/2}"/>
+          <geometry>
+             <cylinder length="${rotation_table_height}" radius="0.27"/>
+          </geometry>
+        </collision>
     </link>
     <joint name="workcell_joint" type="fixed">

Commit message: random

File: hotspray_description/urdf/hotspray_application.xacro (robot description, xacro)
@@ -52,5 +52,5 @@
         <parent link="world"/>
         <child link="tsdf_origin"/>
-      <origin  xyz="0.25 0.25 0.55" rpy="0 0 0" />
+      <origin  xyz="0.2 0.2 0.55" rpy="0 0 0" />
     </joint>
   <!-- tool -->
@@ -62,5 +62,5 @@
     <xacro:include filename="$(find hotspray_description)/urdf/coil_fixed.xacro"/>
       <xacro:coil parent="base_link">
-        <origin  xyz="0.0 0.65 0.1" rpy="0 0 0.0" />
+        <origin  xyz="0.0 0.5 0.1" rpy="0 0 0.0" />
       </xacro:coil>
     </xacro:if>

File: hotspray_description/urdf/hotspray_extruder.xacro (robot description, xacro)
@@ -2,5 +2,5 @@
 <robot xmlns:xacro="http://www.ros.org/wiki/xacro">
   <!-- <xacro:property name="deg_to_rad" value="0.01745329251994329577" /> -->
-  <xacro:macro name="hotspray_extruder" params="parent *origin spray_distance:=${'0.1'}">
+  <xacro:macro name="hotspray_extruder" params="parent *origin spray_distance:=${'0.15'}">
       <!-- extruder_link -->
     <link name="extruder_link"/>

File: hotspray_description/urdf/hotspray_workcell.xacro (robot description, xacro)
@@ -66,5 +66,5 @@
         </collision> -->
     <!-- rotation table collision-->
-        <xacro:property name="rotation_table_height" value="0.1"/>
+        <xacro:property name="rotation_table_height" value="0.05"/>
         <collision>
           <origin rpy="0 0 0" xyz="0.35 0.35 ${table_height + rotation_table_height/2}"/>
