Commit message: egal

File: hotspray_description/urdf/hotspray_workcell.xacro (robot description, xacro)
@@ -79,4 +79,7 @@
       <child link="hotspray_workcell_center"/>
     </joint>
+    <gazebo reference="hotspray_workcell_center">
+      <material>Gazebo/Grey</material>
+    </gazebo>
   </xacro:macro>
 </robot>
