Commit message: motion raster server

File: hotspray_description/urdf/camera/_d435.gazebo.xacro (robot description, xacro)
@@ -132,5 +132,5 @@
       	<rangeMaxDepth>10.0</rangeMaxDepth>
       	<pointCloud>true</pointCloud>
-      	<pointCloudCutoff>0.15</pointCloudCutoff>
+      	<pointCloudCutoff>0.05</pointCloudCutoff>
       	<pointCloudTopicName>/point_cloud</pointCloudTopicName>
       </plugin>

File: hotspray_description/urdf/coil_fixed.xacro (robot description, xacro)
@@ -14,5 +14,5 @@
         <origin xyz="-0.03 0.00 0.02" rpy="1.5708 0 0.0"/>
           <geometry>
-              <mesh filename="package://hotspray_description/meshes/coil.stl" scale="0.001 0.001 0.001" />
+              <mesh filename="package://hotspray_description/meshes/coil.stl" scale="0.0008 0.0008 0.0008" />
           </geometry>
           <material name="orange"/>
@@ -21,5 +21,5 @@
         <origin xyz="-0.03 0.00 0.02" rpy="1.5708 0 0.0"/>
           <geometry>
-              <mesh filename="package://hotspray_description/meshes/coil.stl" scale="0.001 0.001 0.001" />
+              <mesh filename="package://hotspray_description/meshes/coil.stl" scale="0.0008 0.0008 0.0008" />
           </geometry>
       </collision>

File: hotspray_description/urdf/hotspray_application.xacro (robot description, xacro)
@@ -2,5 +2,5 @@
 <robot xmlns:xacro="http://www.ros.org/wiki/xacro" name="hotspray_description">
   <xacro:property name="sim" default="true"/>
-  <xacro:property name="joint_limited" default="false"/>
+  <xacro:property name="joint_limited" default="true"/>
   <xacro:property name="prefix" value=""/>
   <xacro:arg name="transmission_hw_interface" default="hardware_interface/PositionJointInterface" />
@@ -62,5 +62,5 @@
     <xacro:include filename="$(find hotspray_description)/urdf/coil_fixed.xacro"/>
       <xacro:coil parent="base_link">
-        <origin  xyz="0.0 0.6 0.1" rpy="0 0 0.0" />
+        <origin  xyz="0.0 0.65 0.1" rpy="0 0 0.0" />
       </xacro:coil>
     </xacro:if>

File: hotspray_description/urdf/hotspray_camera.xacro (robot description, xacro)
@@ -24,5 +24,5 @@
         <parent link="camera_link"/>
       <child link="camera_orbit_frame"/>
-        <origin xyz="0.25 0.0 0.0" rpy="${-pi/4} ${-pi/2} 0"/>
+        <origin xyz="0.20 0.0 0.0" rpy="${-pi/4} ${-pi/2} 0"/>
     </joint>
   </xacro:macro>

File: hotspray_description/urdf/hotspray_workcell.xacro (robot description, xacro)
@@ -31,38 +31,38 @@
         </inertial>
     <!-- top -->
-        <collision>
+        <!-- <collision>
           <origin rpy="0 0 0" xyz="${offset} ${offset} ${table_height + workspace_height + wall_width/2}"/>
           <geometry>
              <box size="${workspace_width} ${workspace_width} ${wall_width}"/>
           </geometry>
-        </collision>
+        </collision> -->
     <!-- front -->
-        <collision>
+        <!-- <collision>
           <origin rpy="0 0 0" xyz="${offset} ${offset - workspace_width/2 - wall_width/2} ${table_height + workspace_height/2}"/>
           <geometry>
              <box size="${workspace_width} ${wall_width} ${workspace_height}"/>
           </geometry>
-        </collision>
+        </collision> -->
     <!-- back -->
-        <collision>
+        <!-- <collision>
           <origin rpy="0 0 0" xyz="${offset} ${offset + workspace_width/2 + wall_width/2} ${table_height + workspace_height/2}"/>
           <geometry>
              <box size="${workspace_width} ${wall_width} ${workspace_height}"/>
           </geometry>
-        </collision>
+        </collision> -->
     <!-- left -->
-        <collision>
+        <!-- <collision>
           <origin rpy="0 0 0" xyz="${offset - workspace_width/2 - wall_width/2} ${offset} ${table_height + workspace_height/2}"/>
           <geometry>
              <box size="${wall_width} ${workspace_width} ${workspace_height}"/>
           </geometry>
-        </collision>
+        </collision> -->
     <!-- right -->
-        <collision>
+        <!-- <collision>
           <origin rpy="0 0 0" xyz="${offset + workspace_width/2 + wall_width/2} ${offset} ${table_height + workspace_height/2}"/>
           <geometry>
              <box size="${wall_width} ${workspace_width} ${workspace_height}"/>
           </geometry>
-        </collision>
+        </collision> -->
     <!-- rotation table collision-->
         <xacro:property name="rotation_table_height" value="0.1"/>

Commit message: random

File: hotspray_description/urdf/camera/_d435.gazebo.xacro (robot description, xacro)
@@ -129,5 +129,5 @@
       	<infrared1OpticalframeName>${infrared1_optical_frame}</infrared1OpticalframeName>
       	<infrared2OpticalframeName>${infrared2_optical_frame}</infrared2OpticalframeName>
-      	<rangeMinDepth>0.2</rangeMinDepth>
+      	<rangeMinDepth>0.1</rangeMinDepth>
       	<rangeMaxDepth>10.0</rangeMaxDepth>
       	<pointCloud>true</pointCloud>

File: hotspray_description/urdf/hotspray_extruder.xacro (robot description, xacro)
@@ -46,7 +46,7 @@
       </joint> -->
     <!-- joint between fixture and hotspray -->
-       <joint name="hotspray_extruder_joint" type="fixed">
+      <joint name="hotspray_extruder_joint" type="fixed">
         <parent link="${parent}" />
-      <child link="hotspray_extruder" />
+          <child link="hotspray_extruder" />
         <xacro:insert_block name="origin"/>
       </joint>

File: hotspray_description/urdf/hotspray_tool.xacro (robot description, xacro)
@@ -12,8 +12,28 @@
         <xacro:insert_block name="origin"/>
       </joint>
+    <link name="hotspray_adapter">
+      <!-- <inertial>
+        <origin  xyz="0.0 0.0 0.0" rpy="0.0 0.0 0.0" />
+        <mass value="0.0" />
+        <inertia ixx="0.0" ixy="0.0" ixz="0.0" iyy="0.0" iyz="0.0" izz="0.0" />
+      </inertial> -->
+      <visual>
+        <origin  xyz="-0.02 0 0.02" rpy="0 0 0" />
+          <geometry>
+            <box size="0.11 0.015 0.04"/>
+          </geometry>
+        <material name="">
+          <color rgba="0.8 0.8 0.9 1" />
+        </material>
+      </visual>
+      </link>
+      <joint name="hotspray_adapter_joint" type="fixed">
+        <parent link="${parent}"/>
+        <child link="hotspray_adapter"/>
+      </joint>
     <!-- camera -->
       <!-- origin xyz="-0.035 -0.07 0.055" rpy="${-pi/2} ${-pi/2} ${pi/2}"  -->
     <xacro:hotspray_camera parent="hotspray_tool_link" sim="${sim}">
-      <origin xyz="0.03 0.0 0.05" rpy="${pi/2} ${-pi/4} 0" />
+      <origin xyz="0.02 0.014 0.04" rpy="${pi/2} ${-pi/4} 0" />
     </xacro:hotspray_camera>
     <!-- extruder -->
@@ -24,5 +44,5 @@
       <!-- <origin xyz="-0.1 -0.04 0.04" rpy="${-pi/3} 0 ${pi}" /> -->
       <!-- in y direction -->
-      <origin xyz="-0.1 -0.04 0.04" rpy="${-pi/2} 0 ${pi}" />
+      <origin xyz="-0.08 0.0 0.04" rpy="${-pi/2} 0 ${pi}" />
       <!-- in z direction -->
       <!-- <origin xyz="-0.1 -0.04 0.04" rpy="0 0 ${pi}" /> -->
